File: smps.kicad_pcb (KiCad board)
At the start: 2 copper layers, 83.9 x 44 mm, 36 parts, among them J1 Screw_Terminal_01x02, J4 Screw_Terminal_01x02, U1 LT8640S

Commit message: Update PCB layout
Parts:
- moved J1 23.5 mm to (190.5, 124.7), turned to 0 degrees
- moved J4 20.6 mm to (195.5, 96.7), turned to 180 degrees
- moved H4 17.6 mm to (145.6, 128.4)
- moved H3 17.2 mm to (145.6, 93.5)
- moved H2 15.5 mm to (203.5, 128.4)
- moved H1 13.5 mm to (203.5, 93.5)
- moved C2 0.87 mm to (194.4, 109.2), turned to -90 degrees
- moved C3 0.64 mm to (185.3, 109.2), turned to -90 degrees
Routing:
- net +12V: track 36.0 -> 12.1 mm
- net +24V: track 22.3 -> 39.3 mm
- net /L2-L3: track 39.7 -> 37.4 mm
- net GND: vias 36 -> 37
- removed copper zone on F.Cu, net +24V
Other:
- board size 83.9 x 44 mm -> 67 x 44 mm
- board text added: "VIN"
- board text removed: "24V"

Commit message: Cosmetic updates
Parts:
- H1, H2, H3, H4: footprint MountingHole:MountingHole_3.2mm_M3_Pad -> MountingHole:MountingHole_3.2mm_M3
- renumbered TP2 to TP1, TP1 to TP2
Routing:
- net GND: vias 37 -> 38
